Commit message: vat can chuyen dong va chay theo route

File: src/robot_simulation/urdf/robot_core.xacro (robot description, xacro)
@@ -32,5 +32,5 @@
                 <box size="0.3 0.3 0.15"/>
             </geometry>
-            <material name="orange"/>
+            <material name="white"/>
         </visual>
         <collision>
